File: KiCad/BMS_MASTER_25_V0.0.kicad_sch (KiCad schematic)
At the start: 0 parts

Commit message: f
Parts:
- added F1: Fuse, Fuse:Fuseholder_Clip-5x20mm_Eaton_1A5601-01_Inline_P20.80x6.76mm_D1.70mm_Horizontal, symbol Device:Fuse
- added J1, J2, J3: Conn_01x02_Socket, Connector_Molex:Molex_Micro-Fit_3.0_43650-0215_1x02_P3.00mm_Vertical, symbol Connector:Conn_01x02_Socket
Connections:
- new net: F1.1, J1.1 (Pin_1), J1.2 (Pin_2), J2.2 (Pin_2)
- new net HV+: F1.2
- new net HV-: J2.1 (Pin_1), J3.1 (Pin_1), J3.2 (Pin_2)
